File: FR4_Plate_Bottom/Arisutea_FR4_Plate_Bottom.kicad_pcb (KiCad board)
At the start: 2 copper layers, 339.1 x 121 mm, 10 parts

Commit message: Updated plates for copper and logo
Parts:
- removed the G*** at (283.9, 125.8)
- removed the G*** at (284.0, 125.9)
- added G***: LOGO, arisutea:arisutea_logo_mask, F.Cu at (285.0, 129.4)
- added G***: LOGO, arisutea:arisutea_logo_mask, B.Cu at (285.0, 129.4)
- added G***: LOGO, arisutea:arisutea_logo_copper, F.Cu at (285.0, 129.4)
- added G***: LOGO, arisutea:arisutea_logo_copper, B.Cu at (285.0, 129.4)
- added G***: LOGO, arisutea:mattyams_logo_copper, B.Cu at (285.0, 119.9)
- added G***: LOGO, arisutea:mattyams_logo_mask, B.Cu at (285.0, 119.9)
- added G***: LOGO, arisutea:mattyams_logo_copper, F.Cu at (285.0, 119.9)
- added G***: LOGO, arisutea:mattyams_logo_mask, F.Cu at (285.0, 119.9)
Routing:
- added copper zone on B.Cu, net (none)
- added copper zone on F.Cu, net (none)
