File: FR4_Plate_Top/Arisutea_FR4_Plate_Top.kicad_pcb (KiCad board)
At the start: 2 copper layers, 339.1 x 121 mm, 9 parts

Commit message: Updated plates for copper and logo
Parts:
- removed the G*** at (284.0, 125.9)
- added G***: LOGO, arisutea:mattyams_logo_copper, B.Cu at (285.8, 123.8)
- added G***: LOGO, arisutea:mattyams_logo_mask, B.Cu at (285.8, 123.8)
- added G***: LOGO, arisutea:mattyams_logo_mask, F.Cu at (285.8, 123.8)
- added G***: LOGO, arisutea:mattyams_logo_copper, F.Cu at (285.8, 123.8)
- added G***: LOGO, arisutea:arisutea_logo_copper, B.Cu at (285.8, 133.3)
- added G***: LOGO, arisutea:arisutea_logo_mask, B.Cu at (285.8, 133.3)
- added G***: LOGO, arisutea:arisutea_logo_mask, F.Cu at (285.8, 133.3)
- added G***: LOGO, arisutea:arisutea_logo_copper, F.Cu at (285.8, 133.3)
Routing:
- added copper zone on B.Cu, net (none)
- added copper zone on F.Cu, net (none)
