File: FR4_Plate_Top/Arisutea_FR4_Plate_Top.kicad_pcb (KiCad board)
At the start: 2 copper layers, 339.1 x 121 mm, 16 parts

Commit message: added winkey to top fr4 plate
Other:
- outline, holes or cut-outs redrawn
- net class Default removed
